File: boardout.kicad_pcb (KiCad board)
At the start: 2 copper layers, 167.2 x 159.2 mm, 3 parts

Commit message: Initial attempt at connecting connector to circuits. Currently many errors.
Other:
- net class Default removed
