File: hellen154vag-9.1.kicad_pcb (KiCad board)
At the start: 2 copper layers, 164 x 118 mm, 63 parts, among them J1 USB_B_Mini, M1 Module-can-0.1, M2 Module-power5-0.1, M3 Module-mcu-0.1, M4 Module-input-0.1, M5 Module-knock-0.1, M6 Module-output-0.1, M7 Module-ign8-0.1, M8 Module-power12-0.1, P1 368255-2

Commit message: Added 33816 sub schematic changed 121 connector to 154 connector Initial draft schematic. Many nets are not properly connected.
Parts:
- moved C1 35.6 mm to (119.8, 46.4)
- moved D1 35.6 mm to (121.5, 100.4)
- moved F1 35.6 mm to (169.8, 116.8)
- moved F2 35.6 mm to (172.7, 116.8)
- moved J1 35.6 mm to (127.2, 43.7)
- moved M1 35.6 mm to (85.2, 48.7)
- moved M2 35.6 mm to (133.2, 54.4)
- moved M4 35.6 mm to (85.0, 102.4)
- moved M5 35.6 mm to (64.3, 90.4)
- moved M6 35.6 mm to (140.8, 102.0)
- moved M7 35.6 mm to (72.4, 62.5)
- moved M8 35.6 mm to (120.8, 103.3)
- moved P1 35.6 mm to (60.2, 68.5)
- moved R1 35.6 mm to (124.6, 100.3)
- moved R2 35.6 mm to (92.0, 117.9)
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Other:
- outline, holes or cut-outs redrawn
- board text added: "Hellen154vag"
- board text added: "http://rusefi.com/s/hellen154vag"
- board text removed: "Hellen121vag"
- board text removed: "http://rusefi.com/s/hellen121vag"
- board text removed: "© andreika, 2021"

Commit message: Initial attempt at connecting connector to circuits. Currently many errors.
Parts:
- added G?: LOGO, rusefi:LOGO, F.Cu at (67.2, 36.9)
- added G?: Disclaimer, rusefi:Off_Road_Disclaimer, B.Cu at (67.2, 52.1)
- added G?: LOGO, rusefi:LOGO, B.Cu at (67.2, 36.9)
- moved V12 182.8 mm to (296.2, 142.6)
- moved V14 182.8 mm to (290.7, 142.6)
- moved V20 182.8 mm to (278.2, 137.9)
- moved V61 182.8 mm to (267.6, 137.9)
- moved V74 182.8 mm to (272.8, 137.9)
- moved V80 182.8 mm to (262.5, 137.9)
- moved VIN2 182.8 mm to (280.4, 129.1)
- moved VIN3 182.8 mm to (277.6, 129.1)
- moved VIN4 182.8 mm to (274.7, 129.1)
- moved F2 182.8 mm to (353.9, 141.3)
- moved M1 182.8 mm to (266.4, 73.3)
- moved M2 182.8 mm to (314.4, 78.9)
- moved M4 182.8 mm to (266.2, 126.9)
- moved M5 182.8 mm to (245.5, 115.0)
- moved M7 182.8 mm to (253.6, 87.0)
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Other:
- board size 164 x 118 mm -> 357 x 159.2 mm
- board text added: "rusEFI.com"
