File: hellen154vag-9.1.kicad_sch (KiCad schematic)
At the start: 300 parts, among them J1 USB_B_Mini, J10 AudioJack_THR, J2 Conn_01x01, J3 Conn_01x01, J4 Conn_01x01, J5 Conn_01x01, J6 Conn_01x01, J7 Conn_01x04, J8 Conn_01x06, J9 Conn_01x04, M1 Module-can-0.1, M10 Module-can-0.1, M11 Module-vr-0.1, M12 Module-dinput4-0.1, M2 Module-power5-0.2, M3 Module-mcu-0.1, M4 Module-input-0.1, M5 Module-knock-0.1, M6 Module-output-0.1, M7 Module-ign8-0.1, M8 Module-power12-0.1, M9 Module-wbo-0.1, P1 368255-2, U1 L6205PD, U2 LPS25HB, U3 MCP6002-xSN

Commit message: Connected DI IO to E20 and E24. Deleted unused schematic pieces, should be ready for PCB layout. https://github.com/rusefi/hellen154vag-9.1/issues/4
Parts:
- removed F1, F2: Fuse-Pad-Pad, hellen-one-common:PAD-1206-PAD, symbol hellen-one-common:Fuse-Pad-Pad
- removed P1: 368255-2, hellen121vag:368255-2, symbol 368255-2:368255-2
- removed R10, R11, R12, R13, R2, R3, R4, R8, R9: Jumper-Pad-Pad, hellen-one-common:PAD-0805-PAD, symbol hellen-one-common:Jumper-Pad-Pad
- removed V10, V11, V12, V13, V14, V17, V20, V28, V40, V41, V43, V44, V45, V46, V48, V49, V56, V61, V63, V64, V66, V67, V68, V69, V74, V80, V9: Pad, hellen-one-common:PAD-TH, symbol hellen-one-common:Pad
- added W? (x3): TEST, rusEFI_Lib:SM0805_jumper, symbol hellen-one-common:TEST
Connections:
- net TBD_PD3_or_PC13 is gone; now on net E24: W?.2
- net TBD_PD4_or_PA15 is gone; now on net E20: W?.1
- net E20: now reaches M3.E20 (OUT_IO11)
- net E24: now reaches M3.E24 (OUT_IO13)
- net at M3.N25 (SWCLK): now also W?.1
- net at M3.N26 (SWDIO): now also W?.1
- net at M3.N27 (SWO): now also W?.1
- no-connect marks 79 -> 61

Commit message: Changed to pull down resistor, removed series resistor. https://github.com/rusefi/hellen154vag-9.1/issues/6
Parts:
- R5: value 100k -> 10k; LCSC C25803 -> C17513
Connections:
- net ETB_EN: now also C5.2, U1.16 (ENB), U1.5 (ENA)
- net GND: now also R5.2
Other:
- moved on the sheet: R5
Changed lines of the file:
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@@
   (junction (at 323.85 452.755) (diameter 1.016) (color 0 0 0 0))
   (junction (at 326.39 470.535) (diameter 1.016) (color 0 0 0 0))
+  (junction (at 326.39 480.695) (diameter 1.016) (color 0 0 0 0))
   (junction (at 331.47 429.895) (diameter 1.016) (color 0 0 0 0))
+  (junction (at 334.01 470.535) (diameter 1.016) (color 0 0 0 0))
   (junction (at 340.36 429.895) (diameter 1.016) (color 0 0 0 0))
   (junction (at 350.52 429.895) (diameter 1.016) (color 0 0 0 0))
@@
   (no_connect (at 330.2 169.545))
   (no_connect (at 330.2 179.705))
-  (no_connect (at 330.2 187.325))
-  (no_connect (at 330.2 189.865))
+  (no_connect (at 340.36 187.325))
+  (no_connect (at 340.36 189.865))
   (no_connect (at 340.36 192.405))
   (no_connect (at 344.805 172.085))
@@
     (stroke (width 0) (type solid) (color 0 0 0 0))
   )
+  (wire (pts (xy 326.39 470.535) (xy 334.01 470.535))
+    (stroke (width 0) (type solid) (color 0 0 0 0))
+  )
+  (wire (pts (xy 326.39 478.155) (xy 326.39 480.695))
+    (stroke (width 0) (type solid) (color 0 0 0 0))
+  )
+  (wire (pts (xy 326.39 480.695) (xy 334.01 480.695))
+    (stroke (width 0) (type solid) (color 0 0 0 0))
+  )
   (wire (pts (xy 327.66 442.595) (xy 320.04 442.595))
     (stroke (width 0) (type solid) (color 0 0 0 0))
@@
     (stroke (width 0) (type solid) (color 0 0 0 0))
   )
+  (wire (pts (xy 334.01 470.535) (xy 351.79 470.535))
+    (stroke (width 0) (type solid) (color 0 0 0 0))
+  )
   (wire (pts (xy 334.645 149.225) (xy 330.2 149.225))
     (stroke (width 0) (type solid) (color 0 0 0 0))
@@
     (stroke (width 0) (type solid) (color 0 0 0 0))
   )
-  (wire (pts (xy 351.79 470.535) (xy 336.55 470.535))
-    (stroke (width 0) (type solid) (color 0 0 0 0))
-  )
   (wire (pts (xy 359.41 429.895) (xy 351.79 429.895))
     (stroke (width 0) (type solid) (color 0 0 0 0))
@@
     (stroke (width 0) (type solid) (color 0 0 0 0))
   )
-  (bus (pts (xy -13.97 366.395) (xy 62.23 366.395))
-    (stroke (width 0.3048) (type solid) (color 0 255 255 1))
-  )
   (bus (pts (xy 68.58 46.355) (xy 68.58 330.835))
     (stroke (width 0.3048) (type solid) (color 0 0 255 1))
@@
     (pin "1")
   )
-  (symbol (lib_name "power:GND_3") (lib_id "power:GND") (at 326.39 478.155 0) (unit 1)
+  (symbol (lib_name "power:GND_3") (lib_id "power:GND") (at 326.39 480.695 0) (unit 1)
     (in_bom yes) (on_board yes)
-    (property "Reference" "#PWR010" (id 0) (at 326.39 484.505 0)
+    (property "Reference" "#PWR010" (id 0) (at 326.39 487.045 0)
       (effects (font (size 1.27 1.27)) hide)
     )
-    (property "Value" "GND" (id 1) (at 326.4408 482.0984 0))
-    (property "Footprint" "" (id 2) (at 326.39 478.155 0)
+    (property "Value" "GND" (id 1) (at 326.4408 484.6384 0))
+    (property "Footprint" "" (id 2) (at 326.39 480.695 0)
       (effects (font (size 1.27 1.27)) hide)
     )
-    (property "Datasheet" "" (id 3) (at 326.39 478.155 0)
+    (property "Datasheet" "" (id 3) (at 326.39 480.695 0)
       (effects (font (size 1.27 1.27)) hide)
     )
@@
     (pin "2")
   )
-  (symbol (lib_id "hellen-one-common:Res") (at 336.55 470.535 0) (mirror y) (unit 1)
+  (symbol (lib_id "hellen-one-common:Res") (at 334.01 470.535 90) (mirror x) (unit 1)
     (in_bom yes) (on_board yes)
-    (property "Reference" "R5" (id 0) (at 332.74 467.5948 0))
-    (property "Value" "100k" (id 1) (at 331.47 473.7035 0))
-    (property "Footprint" "hellen-one-common:R0603" (id 2) (at 332.74 474.345 0)
+    (property "Reference" "R5" (id 0) (at 331.0698 474.345 0))
+    (property "Value" "10k" (id 1) (at 337.1785 475.615 0))
+    (property "Footprint" "hellen-one-common:R0603" (id 2) (at 337.82 474.345 0)
       (effects (font (size 1.27 1.27)) hide)
     )
-    (property "Datasheet" "" (id 3) (at 336.55 470.535 0)
+    (property "Datasheet" "" (id 3) (at 334.01 470.535 0)
       (effects (font (size 1.27 1.27)) hide)
     )
-    (property "LCSC" "C25803" (id 4) (at 336.55 470.535 0)
+    (property "LCSC" "C17513" (id 4) (at 334.01 470.535 0)
       (effects (font (size 1.27 1.27)) hide)
     )
@@
     )
     (path "/b011732a-563a-40d6-8bbd-df63b18e6dd6"
-      (reference "R5") (unit 1) (value "100k") (footprint "hellen-one-common:R0603")
+      (reference "R5") (unit 1) (value "10k") (footprint "hellen-one-common:R0603")
     )
     (path "/e893da47-8682-43d4-bc9d-8cf03e11db4a"
